File: VFD-disp.kicad_sch (KiCad schematic)
At the start: 118 parts, among them J1 USB_C_Receptacle_USB2.0_14P, J2 Conn_02x03_Odd_Even, J4 Conn_02x03_Odd_Even, J5 Conn_02x03_Odd_Even, J6 Conn_02x03_Odd_Even, Q1 Q_NMOS_GDS, Q2 Q_NMOS_GDS, Q3 Q_NPN_BEC, SW1 SW_SPST, U1 ESP32-C6-WROOM-1, U10 TXS0104EPW, U11 MAX811TEUS-T, U12 MCP4728, U13 TPS2116DRL, U14 KF50BDT, U15 AT24CS01-STUM, U2 FUSB302B01MPX, U3 LM1117DT-3.3, U4 MCP1416, U5 LM2576HVS-ADJ, U6 MAX1771xSA, U7 LM2576HVS-ADJ, U8 USBLC6-2P6, Y1 Crystal

Commit message: wip: values
Parts:
- C1, C14, C17, C19, C2, C26, C29, C3, C30, C33, C36, C4, C5: value C -> 100n
- C27, R25, R26, R7: now not fitted
- C31, C32: value C -> 200-600p
- C34: value C_Polarized -> 1u
- R15, R19: value R -> 100k
- R18, R20: value R -> 1k
- R21, R22, R3, R40, R41: value R -> 4.7k
- R4: value R -> r
Changed lines of the file:
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@@
 		(on_board yes)
 		(in_pos_files yes)
-		(dnp no)
+		(dnp yes)
 		(fields_autoplaced yes)
 		(property "Reference" "R25"
@@
 		(fields_autoplaced yes)
 		(property "Reference" "C3"
-			(at 331.851 108.0078 0)
+			(at 332.74 107.9499 0)
 			(show_name no)
 			(do_not_autoplace no)
@@
 			)
 		)
-		(property "Value" "C"
-			(at 331.851 110.4321 0)
+		(property "Value" "100n"
+			(at 332.74 110.4899 0)
 			(show_name no)
 			(do_not_autoplace no)
@@
 		(fields_autoplaced yes)
 		(property "Reference" "C36"
-			(at 129.921 207.0678 0)
+			(at 130.81 207.0099 0)
 			(show_name no)
 			(do_not_autoplace no)
@@
 			)
 		)
-		(property "Value" "C"
-			(at 129.921 209.4921 0)
+		(property "Value" "100n"
+			(at 130.81 209.5499 0)
 			(show_name no)
 			(do_not_autoplace no)
@@
 		(fields_autoplaced yes)
 		(property "Reference" "C31"
-			(at 75.311 238.8178 0)
+			(at 76.2 238.7599 0)
 			(show_name no)
 			(do_not_autoplace no)
@@
 			)
 		)
-		(property "Value" "C"
-			(at 75.311 241.2421 0)
+		(property "Value" "200-600p"
+			(at 76.2 241.2999 0)
 			(show_name no)
 			(do_not_autoplace no)
@@
 		(on_board yes)
 		(in_pos_files yes)
-		(dnp no)
+		(dnp yes)
 		(property "Reference" "C27"
 			(at 103.251 85.1478 0)
@@
 		(fields_autoplaced yes)
 		(property "Reference" "R4"
-			(at 268.478 360.7378 0)
+			(at 269.24 360.6799 0)
 			(show_name no)
 			(do_not_autoplace no)
@@
 			)
 		)
-		(property "Value" "R"
-			(at 268.478 363.1621 0)
+		(property "Value" "r"
+			(at 269.24 363.2199 0)
 			(show_name no)
 			(do_not_autoplace no)
@@
 		(fields_autoplaced yes)
 		(property "Reference" "U5"
-			(at 245.11 290.4955 0)
+			(at 245.11 289.56 0)
 			(show_name no)
 			(do_not_autoplace no)
@@
 		)
 		(property "Value" "LM2576HVS-ADJ"
-			(at 245.11 292.9198 0)
+			(at 245.11 292.1 0)
 			(show_name no)
 			(do_not_autoplace no)
@@
 		(fields_autoplaced yes)
 		(property "Reference" "C30"
-			(at 278.511 97.8478 0)
+			(at 279.4 97.7899 0)
 			(show_name no)
 			(do_not_autoplace no)
@@
 			)
 		)
-		(property "Value" "C"
-			(at 278.511 100.2721 0)
+		(property "Value" "100n"
+			(at 279.4 100.3299 0)
 			(show_name no)
 			(do_not_autoplace no)
@@
 			)
 		)
-		(property "Value" "C"
+		(property "Value" "100n"
 			(at 83.82 217.1699 0)
 			(show_name no)
@@
 		(on_board yes)
 		(in_pos_files yes)
-		(dnp no)
+		(dnp yes)
 		(fields_autoplaced yes)
 		(property "Reference" "R26"
@@
 		(fields_autoplaced yes)
 		(property "Reference" "C5"
-			(at 215.011 360.7378 0)
+			(at 215.9 360.6799 0)
 			(show_name no)
 			(do_not_autoplace no)
@@
 			)
 		)
-		(property "Value" "C"
-			(at 215.011 363.1621 0)
+		(property "Value" "100n"
+			(at 215.9 363.2199 0)
 			(show_name no)
 			(do_not_autoplace no)
@@
 		(fields_autoplaced yes)
 		(property "Reference" "R15"
-			(at 113.538 115.6278 0)
+			(at 114.3 115.5699 0)
 			(show_name no)
 			(do_not_autoplace no)
@@
 			)
 		)
-		(property "Value" "R"
-			(at 113.538 118.0521 0)
+		(property "Value" "100k"
+			(at 114.3 118.1099 0)
 			(show_name no)
 			(do_not_autoplace no)
@@
 		(fields_autoplaced yes)
 		(property "Reference" "C33"
-			(at 460.121 157.5378 0)
+			(at 461.01 157.4799 0)
 			(show_name no)
 			(do_not_autoplace no)
@@
 			)
 		)
-		(property "Value" "C"
-			(at 460.121 159.9621 0)
+		(property "Value" "100n"
+			(at 461.01 160.0199 0)
 			(show_name no)
 			(do_not_autoplace no)
@@
 		(fields_autoplaced yes)
 		(property "Reference" "C1"
-			(at 331.851 34.3478 0)
+			(at 332.74 34.2899 0)
 			(show_name no)
 			(do_not_autoplace no)
@@
 			)
 		)
-		(property "Value" "C"
-			(at 331.851 36.7721 0)
+		(property "Value" "100n"
+			(at 332.74 36.8299 0)
 			(show_name no)
 			(do_not_autoplace no)
@@
 		(fields_autoplaced yes)
 		(property "Reference" "C32"
-			(at 85.471 238.8178 0)
+			(at 86.36 238.7599 0)
 			(show_name no)
 			(do_not_autoplace no)
@@
 			)
 		)
-		(property "Value" "C"
-			(at 85.471 241.2421 0)
+		(property "Value" "200-600p"
+			(at 86.36 241.2999 0)
 			(show_name no)
 			(do_not_autoplace no)
@@
 		(fields_autoplaced yes)
 		(property "Reference" "R20"
-			(at 121.158 135.9478 0)
+			(at 121.92 135.8899 0)
 			(show_name no)
 			(do_not_autoplace no)
@@
 			)
 		)
-		(property "Value" "R"
-			(at 121.158 138.3721 0)
+		(property "Value" "1k"
+			(at 121.92 138.4299 0)
 			(show_name no)
 			(do_not_autoplace no)
@@
 		(fields_autoplaced yes)
 		(property "Reference" "C29"
-			(at 127.381 274.3778 0)
+			(at 128.27 274.3199 0)
 			(show_name no)
 			(do_not_autoplace no)
@@
 			)
 		)
-		(property "Value" "C"
-			(at 127.381 276.8021 0)
+		(property "Value" "100n"
+			(at 128.27 276.8599 0)
 			(show_name no)
 			(do_not_autoplace no)
@@
 		(fields_autoplaced yes)
 		(property "Reference" "C26"
-			(at 213.741 64.8278 0)
+			(at 214.63 64.7699 0)
 			(show_name no)
 			(do_not_autoplace no)
@@
 			)
 		)
-		(property "Value" "C"
-			(at 213.741 67.2521 0)
+		(property "Value" "100n"
+			(at 214.63 67.3099 0)
 			(show_name no)
 			(do_not_autoplace no)
@@
 		(fields_autoplaced yes)
 		(property "Reference" "C34"
-			(at 470.281 156.6488 0)
+			(at 471.17 156.5909 0)
 			(show_name no)
 			(do_not_autoplace no)
@@
 			)
 		)
-		(property "Value" "C_Polarized"
-			(at 470.281 159.0731 0)
+		(property "Value" "1u"
+			(at 471.17 159.1309 0)
 			(show_name no)
 			(do_not_autoplace no)
@@
 		(fields_autoplaced yes)
 		(property "Reference" "R40"
-			(at 245.618 99.1178 0)
+			(at 246.38 99.0599 0)
 			(show_name no)
 			(do_not_autoplace no)
@@
 			)
 		)
-		(property "Value" "R"
-			(at 245.618 101.5421 0)
+		(property "Value" "4.7k"
+			(at 246.38 101.5999 0)
 			(show_name no)
 			(do_not_autoplace no)
@@
 			)
 		)
-		(property "Value" "R"
+		(property "Value" "4.7k"
 			(at 486.41 325.1199 0)
 			(show_name no)
@@
 			)
 		)
-		(property "Value" "R"
+		(property "Value" "4.7k"
 			(at 429.26 325.1199 0)
 			(show_name no)
@@
 		(fields_autoplaced yes)
 		(property "Reference" "R18"
-			(at 113.538 123.2478 0)
+			(at 114.3 123.1899 0)
 			(show_name no)
 			(do_not_autoplace no)
@@
 			)
 		)
-		(property "Value" "R"
-			(at 113.538 125.6721 0)
+		(property "Value" "1k"
+			(at 114.3 125.7299 0)
 			(show_name no)
 			(do_not_autoplace no)
@@
 		(fields_autoplaced yes)
 		(property "Reference" "C4"
-			(at 339.471 108.0078 0)
+			(at 340.36 107.9499 0)
 			(show_name no)
 			(do_not_autoplace no)
@@
 			)
 		)
-		(property "Value" "C"
-			(at 339.471 110.4321 0)
+		(property "Value" "100n"
+			(at 340.36 110.4899 0)
 			(show_name no)
 			(do_not_autoplace no)
@@
 		(fields_autoplaced yes)
 		(property "Reference" "R19"
-			(at 121.158 128.3278 0)
+			(at 121.92 128.2699 0)
 			(show_name no)
 			(do_not_autoplace no)
@@
 			)
 		)
-		(property "Value" "R"
-			(at 121.158 130.7521 0)
+		(property "Value" "100k"
+			(at 121.92 130.8099 0)
 			(show_name no)
 			(do_not_autoplace no)
@@
 		(on_board yes)
 		(in_pos_files yes)
-		(dnp no)
+		(dnp yes)
 		(fields_autoplaced yes)
 		(property "Reference" "R7"
@@
 		(fields_autoplaced yes)
 		(property "Reference" "R3"
-			(at 210.058 341.6878 0)
+			(at 210.82 341.6299 0)
 			(show_name no)
 			(do_not_autoplace no)
@@
 			)
 		)
-		(property "Value" "R"
-			(at 210.058 344.1121 0)
+		(property "Value" "4.7k"
+			(at 210.82 344.1699 0)
 			(show_name no)
 			(do_not_autoplace no)
@@
 		(fields_autoplaced yes)
 		(property "Reference" "C2"
-			(at 339.471 34.3478 0)
+			(at 340.36 34.2899 0)
 			(show_name no)
 			(do_not_autoplace no)
@@
 			)
 		)
-		(property "Value" "C"
-			(at 339.471 36.7721 0)
+		(property "Value" "100n"
+			(at 340.36 36.8299 0)
 			(show_name no)
 			(do_not_autoplace no)
@@
 		(fields_autoplaced yes)
 		(property "Reference" "R41"
-			(at 253.238 99.1178 0)
+			(at 254 99.0599 0)
 			(show_name no)
 			(do_not_autoplace no)
@@
 			)
 		)
-		(property "Value" "R"
-			(at 253.238 101.5421 0)
+		(property "Value" "4.7k"
+			(at 254 101.5999 0)
 			(show_name no)
 			(do_not_autoplace no)
@@
 		(fields_autoplaced yes)
 		(property "Reference" "C19"
-			(at 296.291 97.8478 0)
+			(at 297.18 97.7899 0)
 			(show_name no)
 			(do_not_autoplace no)
@@
 			)
 		)
-		(property "Value" "C"
-			(at 296.291 100.2721 0)
+		(property "Value" "100n"
+			(at 297.18 100.3299 0)
 			(show_name no)
 			(do_not_autoplace no)
@@
 		(fields_autoplaced yes)
 		(property "Reference" "C17"
-			(at 118.491 334.0678 0)
+			(at 119.38 334.0099 0)
 			(show_name no)
 			(do_not_autoplace no)
@@
 			)
 		)
-		(property "Value" "C"
-			(at 118.491 336.4921 0)
+		(property "Value" "100n"
+			(at 119.38 336.5499 0)
 			(show_name no)
 			(do_not_autoplace no)
