File: VFD-disp.kicad_sch (KiCad schematic)
At the start: 118 parts, among them J1 USB_C_Receptacle_USB2.0_14P, J2 Conn_02x03_Odd_Even, J4 Conn_02x03_Odd_Even, J5 Conn_02x03_Odd_Even, J6 Conn_02x03_Odd_Even, Q1 Q_NMOS_GDS, Q2 Q_NMOS_GDS, Q3 Q_NPN_BEC, SW1 SW_SPST, U1 ESP32-C6-WROOM-1, U10 TXS0104EPW, U11 MAX811TEUS-T, U12 MCP4728, U13 TPS2116DRL, U14 KF50BDT, U15 AT24CS01-STUM, U2 FUSB302B01MPX, U3 LM1117DT-3.3, U4 MCP1416, U5 LM2576HVS-ADJ, U6 MAX1771xSA, U7 LM2576HVS-ADJ, U8 USBLC6-2P6, Y1 Crystal

Commit message: values and TME
Parts:
- C1, C17, C19, C2, C26, C29, C3, C30, C33, C36, C4, C5: value 100n -> 100nF
- C10: value C -> Giga cap; now not fitted
- C11, C12, C18, C20, C23, C35, C40, C41: value C -> 100nF
- C13, C21, C22, C24, C25, C6: value C_Polarized -> 150uF; TME_SYMBOL (none) -> EEEFT1A151AR
- C14: value 100n -> 100nF; now not fitted
- C15, C16, Y1: now not fitted
- C28: value C_Polarized -> 40uF; TME_SYMBOL (none) -> T491D476K010AT
- C31, C32: value 200-600p -> 200-600pF
- C34: value 1u -> 40uF; TME_SYMBOL (none) -> T491D476K010AT
- C37, C8, C9: value C -> 100nF; now not fitted
- C38, C39: TME_SYMBOL (none) -> CS3216X5R106M500NR
- C7: value C_Polarized -> 10uF; TME_SYMBOL (none) -> VS1H100MC054000CE0
- D1: value D -> B3100BE-13; TME_SYMBOL (none) -> B3100BE-13
- D2: value D_Zener -> Zener 3.5V
- D3, D4: value D_Schottky -> SS24
- F1: value Fuse -> 2A; TME_SYMBOL (none) -> PTSLR08058V200
- F4: value Fuse -> 500mA; TME_SYMBOL (none) -> 0ZCK0050FF2E
- F5: value Fuse -> 750mA; TME_SYMBOL (none) -> SR075-06
- HV5812WG1, HV5812WG2, IVLM3-5/1: now left out of the parts list
- L1, L3, L4: value L -> 100uH; TME_SYMBOL (none) -> PSDB1004NT101
- R10: value R -> 10
- R11, R12, R16, R29, R6: value R -> 10k
- R17, R30: value R -> 100k
- R24: value R -> 1k
- R4: value r -> 40m
- R5: value R -> ~70k
- RV1: value R_Potentiometer -> 20k
- RV3: value R_Potentiometer -> 100k
- U7: value LM2576HVS-ADJ -> LM2576HVS-0.5
Other:
- note added: "F = 3.1V"
- note added: "Jebać ten kwarc nie ma w TME"
- note added: "VPP <= 27V"
- moved on the sheet: C13, C18, C22, C6, F5, R16, R9, RV1

Commit message: some changes
Parts:
- C1, C10, C11, C12, C15, C16, C17, C18, C19, C2, C20, C23, C26, C27, C29, C3, C30, C33, C35, C36, C37, C4, C40, C41, C5, C8, C9, Q2, R25, R26, R7, R9, Y1: now left out of the parts list
- L1, L3, L4, Q1, U12, U13, U2, U4, U5, U6, U8: Comment (none) -> already have; now left out of the parts list
- R13, R44, R8: now not fitted; now left out of the parts list
- R14: value R -> 10k
- R5: value ~70k -> 130k
- RV3: value 100k -> 20k
- U7: value LM2576HVS-0.5 -> LM2576-5.0WU
Other:
- note added: "BAD ZENER FOOTPRINT"
- note added: "RDY can float if unused"
- note added: "req: VPP <= 27V 150k/10k -> 24V 130k/10k -> 21V"
- note removed: "VPP <= 27V"

Commit message: some resistor values
Parts:
- R23: value R -> 3.83k
- R27: value R -> 1k
- R28: value R -> 4.7k
- R9: value R -> 0R
Changed lines of the file:
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@@
 		(fields_autoplaced yes)
 		(property "Reference" "R28"
-			(at 395.478 251.5178 0)
+			(at 396.24 251.4599 0)
 			(show_name no)
 			(do_not_autoplace no)
@@
 			)
 		)
-		(property "Value" "R"
-			(at 395.478 253.9421 0)
+		(property "Value" "4.7k"
+			(at 396.24 253.9999 0)
 			(show_name no)
 			(do_not_autoplace no)
@@
 		(fields_autoplaced yes)
 		(property "Reference" "R27"
-			(at 343.408 250.2478 0)
+			(at 344.17 250.1899 0)
 			(show_name no)
 			(do_not_autoplace no)
@@
 			)
 		)
-		(property "Value" "R"
-			(at 343.408 252.6721 0)
+		(property "Value" "1k"
+			(at 344.17 252.7299 0)
 			(show_name no)
 			(do_not_autoplace no)
@@
 		(fields_autoplaced yes)
 		(property "Reference" "R23"
-			(at 343.408 240.0878 0)
+			(at 344.17 240.0299 0)
 			(show_name no)
 			(do_not_autoplace no)
@@
 			)
 		)
-		(property "Value" "R"
-			(at 343.408 242.5121 0)
+		(property "Value" "3.83k"
+			(at 344.17 242.5699 0)
 			(show_name no)
 			(do_not_autoplace no)
@@
 		(fields_autoplaced yes)
 		(property "Reference" "R9"
-			(at 331.47 308.5295 90)
+			(at 331.47 307.34 90)
 			(show_name no)
 			(do_not_autoplace no)
@@
 			)
 		)
-		(property "Value" "R"
-			(at 331.47 310.9538 90)
+		(property "Value" "0R"
+			(at 331.47 309.88 90)
 			(show_name no)
 			(do_not_autoplace no)

Commit message: first working code
Parts:
- R9: value 0R -> R; now not fitted
Connections:
- net +3.3V: now also U10.8 (OE)
- net GND: no longer U10.8 (OE)
Changed lines of the file:
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@@
 	)
 	(junction
-		(at 134.62 90.17)
-		(diameter 0)
-		(color 0 0 0 0)
-	)
-	(junction
 		(at 287.02 302.26)
 		(diameter 0)
@@
 	)
 	(junction
+		(at 134.62 82.55)
+		(diameter 0)
+		(color 0 0 0 0)
+	)
+	(junction
 		(at 454.66 287.02)
 		(diameter 0)
@@
 	)
 	(junction
-		(at 469.9 284.48)
+		(at 283.21 105.41)
 		(diameter 0)
 		(color 0 0 0 0)
 	)
 	(junction
-		(at 285.75 134.62)
+		(at 469.9 284.48)
 		(diameter 0)
 		(color 0 0 0 0)
@@
 	)
 	(junction
+		(at 251.46 110.49)
+		(diameter 0)
+		(color 0 0 0 0)
+	)
+	(junction
 		(at 190.5 365.76)
 		(diameter 0)
@@
 	)
 	(junction
-		(at 195.58 227.33)
+		(at 243.84 107.95)
 		(diameter 0)
 		(color 0 0 0 0)
 	)
 	(junction
-		(at 431.8 284.48)
+		(at 195.58 227.33)
 		(diameter 0)
 		(color 0 0 0 0)
 	)
 	(junction
-		(at 251.46 110.49)
+		(at 431.8 284.48)
 		(diameter 0)
 		(color 0 0 0 0)
@@
 	)
 	(junction
-		(at 243.84 107.95)
-		(diameter 0)
-		(color 0 0 0 0)
-	)
-	(junction
 		(at 55.88 237.49)
 		(diameter 0)
@@
 	)
 	(junction
+		(at 134.62 90.17)
+		(diameter 0)
+		(color 0 0 0 0)
+	)
+	(junction
 		(at 229.87 365.76)
 		(diameter 0)
@@
 		(color 0 0 0 0)
 	)
-	(junction
-		(at 134.62 82.55)
-		(diameter 0)
-		(color 0 0 0 0)
-	)
 	(no_connect
 		(at 365.76 74.93)
@@
 	(wire
 		(pts
-			(xy 285.75 134.62) (xy 285.75 130.81)
+			(xy 285.75 130.81) (xy 285.75 137.16)
 		)
 		(stroke
@@
 	(wire
 		(pts
-			(xy 469.9 284.48) (xy 469.9 287.02)
+			(xy 271.78 113.03) (xy 271.78 105.41)
 		)
 		(stroke
@@
 	(wire
 		(pts
-			(xy 227.33 337.82) (xy 234.95 337.82)
+			(xy 469.9 284.48) (xy 469.9 287.02)
 		)
 		(stroke
@@
 	(wire
 		(pts
-			(xy 275.59 113.03) (xy 271.78 113.03)
+			(xy 227.33 337.82) (xy 234.95 337.82)
 		)
 		(stroke
@@
 		)
 	)
-	(bus
+	(wire
 		(pts
-			(xy 466.09 127) (xy 466.09 129.54)
+			(xy 271.78 113.03) (xy 275.59 113.03)
 		)
 		(stroke
@@
 		)
 	)
-	(wire
+	(bus
 		(pts
-			(xy 339.09 57.15) (xy 321.31 57.15)
+			(xy 466.09 127) (xy 466.09 129.54)
 		)
 		(stroke
@@
 	(wire
 		(pts
-			(xy 285.75 134.62) (xy 285.75 137.16)
+			(xy 339.09 57.15) (xy 321.31 57.15)
 		)
 		(stroke
@@
 	(wire
 		(pts
+			(xy 271.78 105.41) (xy 283.21 105.41)
+		)
+		(stroke
+			(width 0)
+			(type default)
+		)
+	)
+	(wire
+		(pts
 			(xy 468.63 93.98) (xy 483.87 93.98)
 		)
@@
 	(wire
 		(pts
-			(xy 271.78 134.62) (xy 285.75 134.62)
-		)
-		(stroke
-			(width 0)
-			(type default)
-		)
-	)
-	(wire
-		(pts
 			(xy 55.88 237.49) (xy 57.15 237.49)
 		)
@@
 	(wire
 		(pts
-			(xy 271.78 113.03) (xy 271.78 134.62)
-		)
-		(stroke
-			(width 0)
-			(type default)
-		)
-	)
-	(wire
-		(pts
 			(xy 356.87 234.95) (xy 365.76 234.95)
 		)
@@
 		(property "Value" "HV5812WG"
 			(at 353.9841 101.8074 0)
+			(hide yes)
 			(show_name no)
 			(do_not_autoplace no)
@@
 		(in_pos_files yes)
 		(dnp no)
-		(fields_autoplaced yes)
 		(property "Reference" "U4"
-			(at 487.8879 166.4734 0)
+			(at 480.568 162.814 0)
 			(show_name no)
 			(do_not_autoplace no)
@@
 		)
 		(property "Value" "MCP1416"
-			(at 487.8879 168.8977 0)
+			(at 480.568 165.1 0)
 			(show_name no)
 			(do_not_autoplace no)
@@
 		(on_board yes)
 		(in_pos_files yes)
-		(dnp no)
+		(dnp yes)
 		(fields_autoplaced yes)
 		(property "Reference" "R9"
@@
 			)
 		)
-		(property "Value" "0R"
+		(property "Value" "R"
 			(at 331.47 309.88 90)
 			(show_name no)

Commit message: update PCB with fixed values
Parts:
- R1, R2: value R -> 0R
- R5: value 130k -> 2.7k
- R6: value 10k -> 1.2k
Other:
- note added: "F = 2.8V"
- note removed: "F = 3.1V"
- note removed: "req: VPP <= 27V 150k/10k -> 24V 130k/10k -> 21V"
- moved on the sheet: R2
Changed lines of the file:
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@@
 	(generator_version "10.0")
 	(paper "A2")
-	(text "req: VPP <= 27V\n150k/10k -> 24V\n130k/10k -> 21V"
-		(exclude_from_sim no)
-		(at 304.292 330.454 0)
-		(effects
-			(font
-				(size 1.27 1.27)
-			)
-		)
-	)
-	(text "F = 3.1V"
+	(text "F = 2.8V"
 		(exclude_from_sim no)
 		(at 338.836 295.402 0)
@@
 	)
 	(junction
-		(at 495.3 154.94)
-		(diameter 0)
-		(color 0 0 0 0)
-	)
-	(junction
 		(at 215.9 60.96)
 		(diameter 0)
@@
 	)
 	(junction
+		(at 491.49 154.94)
+		(diameter 0)
+		(color 0 0 0 0)
+	)
+	(junction
 		(at 433.07 234.95)
 		(diameter 0)
@@
 	(wire
 		(pts
+			(xy 491.49 144.78) (xy 495.3 144.78)
+		)
+		(stroke
+			(width 0)
+			(type default)
+		)
+	)
+	(wire
+		(pts
 			(xy 397.51 234.95) (xy 402.59 234.95)
 		)
@@
 	(wire
 		(pts
-			(xy 495.3 154.94) (xy 497.84 154.94)
-		)
-		(stroke
-			(width 0)
-			(type default)
-		)
-	)
-	(wire
-		(pts
 			(xy 458.47 172.72) (xy 462.28 172.72)
 		)
@@
 	(wire
 		(pts
-			(xy 490.22 154.94) (xy 495.3 154.94)
+			(xy 490.22 154.94) (xy 491.49 154.94)
 		)
 		(stroke
@@
 	(wire
 		(pts
+			(xy 491.49 154.94) (xy 497.84 154.94)
+		)
+		(stroke
+			(width 0)
+			(type default)
+		)
+	)
+	(wire
+		(pts
 			(xy 264.16 74.93) (xy 266.7 74.93)
 		)
@@
 	(wire
 		(pts
-			(xy 495.3 152.4) (xy 495.3 154.94)
+			(xy 491.49 152.4) (xy 491.49 154.94)
 		)
 		(stroke
@@
 		(in_pos_files yes)
 		(dnp no)
-		(fields_autoplaced yes)
 		(property "Reference" "#PWR0104"
 			(at 111.76 116.84 0)
@@
 		)
 		(property "Value" "VPP"
-			(at 111.76 108.8969 0)
+			(at 110.744 108.966 0)
 			(show_name no)
 			(do_not_autoplace no)
@@
 					(size 1.27 1.27)
 				)
+				(justify left)
 			)
 		)
@@
 			)
 		)
-		(property "Value" "130k"
+		(property "Value" "2.7k"
 			(at 298.45 342.8999 0)
 			(show_name no)
@@
 	(symbol
 		(lib_id "Device:R")
-		(at 495.3 148.59 0)
+		(at 491.49 148.59 0)
 		(unit 1)
 		(body_style 1)
@@
 		(fields_autoplaced yes)
 		(property "Reference" "R2"
-			(at 497.078 147.3778 0)
+			(at 494.03 147.3199 0)
 			(show_name no)
 			(do_not_autoplace no)
@@
 			)
 		)
-		(property "Value" "R"
-			(at 497.078 149.8021 0)
+		(property "Value" "0R"
+			(at 494.03 149.8599 0)
 			(show_name no)
 			(do_not_autoplace no)
@@
 		)
 		(property "Footprint" "Resistor_SMD:R_0805_2012Metric"
-			(at 493.522 148.59 90)
+			(at 489.712 148.59 90)
 			(hide yes)
 			(show_name no)
@@
 		)
 		(property "Datasheet" ""
-			(at 495.3 148.59 0)
+			(at 491.49 148.59 0)
 			(hide yes)
 			(show_name no)
@@
 		)
 		(property "Description" "Resistor"
-			(at 495.3 148.59 0)
+			(at 491.49 148.59 0)
 			(hide yes)
 			(show_name no)
@@
 		)
 		(property "TME_SYMBOL" ""
-			(at 495.3 148.59 0)
+			(at 491.49 148.59 0)
 			(hide yes)
 			(show_name no)
@@
 		)
 		(property "Comment" ""
-			(at 495.3 148.59 0)
+			(at 491.49 148.59 0)
 			(hide yes)
 			(show_name no)
@@
 			)
 		)
-		(property "Value" "10k"
+		(property "Value" "1.2k"
 			(at 298.45 363.2199 0)
 			(show_name no)
@@
 		(fields_autoplaced yes)
 		(property "Reference" "R1"
-			(at 499.618 147.3778 0)
+			(at 500.38 147.3199 0)
 			(show_name no)
 			(do_not_autoplace no)
@@
 			)
 		)
-		(property "Value" "R"
-			(at 499.618 149.8021 0)
+		(property "Value" "0R"
+			(at 500.38 149.8599 0)
 			(show_name no)
 			(do_not_autoplace no)

Commit message: Rev 2 of schematic
Parts:
- removed C15, C16: C, Capacitor_SMD:C_0805_2012Metric, symbol Device:C
- removed C25, C6: 150uF, Capacitor_SMD:CP_Elec_5x4.5, symbol Device:C_Polarized
- removed C29, C35, C5: 100nF, Capacitor_SMD:C_0805_2012Metric, symbol Device:C
- removed C34: 40uF, Capacitor_Tantalum_SMD:CP_EIA-7343-31_Kemet-D, symbol Device:C_Polarized
- removed C7: 10uF, Capacitor_SMD:CP_Elec_5x4.5, symbol Device:C_Polarized
- removed C8: 100nF, Capacitor_SMD:C_2220_5750Metric, symbol Device:C
- removed D1: B3100BE-13, Diode_SMD:D_SMB, symbol Device:D
- removed D4: SS24, Diode_SMD:D_SMB, symbol Device:D_Schottky
- removed D6: BZV55B7V5, Diode_SMD:D_MiniMELF, symbol Diode:BZV55B7V5
- removed L1, L4: 100uH, Inductor_SMD:L_Bourns_SRP1038C_10.0x10.0mm, symbol Device:L
- removed Q1: Q_NMOS_GDS, Package_TO_SOT_SMD:TO-263-2, symbol Transistor_FET:Q_NMOS_GDS
- removed Q3: Q_NPN_BEC, Package_TO_SOT_SMD:SOT-23, symbol Transistor_BJT:Q_NPN_BEC
- removed R28, R3: 4.7k, Resistor_SMD:R_0805_2012Metric, symbol Device:R
- removed R29: 10k, Resistor_SMD:R_0805_2012Metric, symbol Device:R
- removed R30: 100k, Resistor_SMD:R_0805_2012Metric, symbol Device:R
- removed R4: 40m, Resistor_SMD:R_0805_2012Metric, symbol Device:R
- removed R44, R8: R, Resistor_SMD:R_0805_2012Metric, symbol Device:R
- removed R5: 2.7k, Resistor_SMD:R_0805_2012Metric, symbol Device:R
- removed R6: 1.2k, Resistor_SMD:R_0805_2012Metric, symbol Device:R
- removed RV3: 20k, Potentiometer_SMD:Potentiometer_Bourns_3269W_Vertical, symbol Device:R_Potentiometer
- removed U12: MCP4728, Package_SO:MSOP-10_3x3mm_P0.5mm, symbol Analog_DAC:MCP4728
- removed U13: TPS2116DRL, Package_TO_SOT_SMD:SOT-583-8, symbol Power_Management:TPS2116DRL
- removed U4: MCP1416, Package_TO_SOT_SMD:SOT-23-5, symbol Driver_FET:MCP1416
- removed U6: MAX1771xSA, Package_SO:SO-8_3.9x4.9mm_P1.27mm, symbol Regulator_Switching:MAX1771xSA
- removed U7: LM2576-5.0WU, Package_TO_SOT_SMD:TO-263-5_TabPin3, symbol Regulator_Switching:LM2576HVS-ADJ
- removed Y1: Crystal, Crystal:Crystal_SMD_HC49-SD, symbol Device:Crystal
- added C15: 10uF, Capacitor_SMD:CP_Elec_5x4.5, symbol Device:C_Polarized
- added C16: 150uF, Capacitor_SMD:CP_Elec_5x4.5, symbol Device:C_Polarized
- added C42: 100nF, Capacitor_SMD:C_0805_2012Metric, symbol Device:C
- added C43: 3.3nF, Capacitor_SMD:C_0805_2012Metric, symbol Device:C
- added C44: 1nF, Capacitor_SMD:C_0805_2012Metric, symbol Device:C
- added D10, D5, D7, D8, D9: BZT52C3V3-7-F, Diode_SMD:D_SOD-123, symbol Device:D_Zener
- added D4: B3100BE-13, Diode_SMD:D_SMB, symbol Device:D
- added L2: 47uF, Inductor_SMD:L_Bourns_SRP1038C_10.0x10.0mm, symbol Device:L
- added R33, R34, R35, R36, R37: 1k, Resistor_SMD:R_0805_2012Metric, symbol Device:R
- added RV4: 20k, Potentiometer_SMD:Potentiometer_Bourns_3269W_Vertical, symbol Device:R_Potentiometer
- added U4: MCP4661-103E_ST, Package_SO:TSSOP-14_4.4x5mm_P0.65mm, symbol JLCImport:MCP4661-103E_ST
- added U7: LM3478MA, Package_SO:SOIC-8_3.9x4.9mm_P1.27mm, symbol Regulator_Controller:LM3478MA
- added U9: DRV8837, Package_SON:WSON-8-1EP_2x2mm_P0.5mm_EP0.9x1.6mm, symbol Driver_Motor:DRV8837
- Q2: Comment (none) -> already have
- R10: value 10 -> 2.7k
- R11: value 10k -> 1.2k
- R12: value 10k -> R; now not fitted; now left out of the parts list
- R13: value R -> 40m; now fitted; now in the parts list
- R14: value 10k -> 26k7
- R17: value 100k -> 10K
- R23: value 3.83k -> 100k
- R27: value 1k -> 56k2
Connections:
- net 4728_RDY is gone; now on net GND: R13.2
- net +3.3V: now also C33.1, U4.14 (VDD), U9.7 (~{SLEEP}), U9.8 (VCC); no longer R13.1
- net +5V: no longer C33.1
- net F: now also U9.1 (VM); no longer R1.2, R2.2
- net F_ADJ: now also U4.7 (P1A)
- net F_EN: now also U9.5 (IN2)
- net F_PWM: now also U9.6 (IN1); no longer R12.1
- net G1: now also D5.1 (K), R33.2; no longer HV5812WG2.11 (OUT12)
- net G2: now also D7.1 (K), R34.2; no longer HV5812WG2.10 (OUT13)
- net G3: now also D8.1 (K), R36.2; no longer HV5812WG2.9 (OUT14)
- net G4: now also D9.1 (K), R35.2; no longer HV5812WG2.8 (OUT15)
- net G5: now also D10.1 (K), R37.2; no longer HV5812WG2.7 (OUT16)
- net GND: now also R24.2, C16.2, C42.2, C44.2, D10.2 (A), D5.2 (A), D7.2 (A), D8.2 (A), D9.2 (A), U4.1 (HVC/A0), U4.12 (A2), U4.13 (A1), U4.4 (VSS), U4.6 (P1W), U4.9 (P0W), U7.4 (AGND), U7.5 (PGND), U9.4 (GND), U9.9 (GND); no longer C9.2, Q2.3 (S), R11.2, R12.2
- net HV_ADJ: now also R12.2, U4.8 (P0A)
- net SCL: now also U4.2 (SCL)
- net SDA: now also U4.3 (SDA)
- net VBUS: now also R23.1, C16.1, C42.1, L2.1, U7.8 (V_{IN}); no longer C23.1, R24.1
- net VPP: now also C9.1, R10.1, C15.1, D4.1 (K)
- net at C39.1, C41.1, U14.3 (VO): now also F4.1
- net at U1.9 (GPIO1/ADC1_CH1/XTAL_32K_N): now also C23.1, R23.2, R24.1
- net at R27.1: now also C43.2, C44.1; no longer R23.2
- net at Q2.2 (D): now also D4.2 (A), L2.2; no longer IVLM3-5/1.22 (F2)
- net NEG_LDAC: no longer names the net of R14.1
- net NEG_LDAC: now also U7.7 (FA/SD)
- new net: Q2.1 (G), U7.6 (DR)
- new net: Q2.3 (S), R13.1, U7.1 (I_{SEN})
- new net: R11.1, R12.1, RV4.2, U7.3 (FB)
- new net: C15.2, C9.2, R11.2
- new net: HV5812WG2.9 (OUT14), R36.1
- new net: HV5812WG2.11 (OUT12), R33.1
- new net: HV5812WG2.8 (OUT15), R35.1
- new net: R10.2, RV4.1
- new net: HV5812WG2.10 (OUT13), R34.1
- new net: IVLM3-5/1.22 (F2), U9.3 (OUT2)
- new net: HV5812WG2.7 (OUT16), R37.1
- new net: C43.1, U7.2 (COMP)
- new net: R1.2, R2.2, U9.2 (OUT1)
- no-connect marks 16 -> 20
Other:
- note removed: "RDY can float if unused"
- moved on the sheet: C10, C11, C12, C13, C38, C39, C40, C41, F4, R17, U14, U3

Commit message: run autoroute
Parts:
- C1, C11, C12, C17, C18, C19, C2, C20, C23, C26, C3, C30, C33, C36, C4, C40, C41, C42, C9: LCSC (none) -> C7419429
- C13, C14, C15, C16, C21, C22, C24, C27, C28, C31, C32, C37, C38, C39, C43, C44, D2, D4, D5, F1, F4, F5, H1, H2, HV5812WG1, HV5812WG2, IVLM3-5/1, J1, J2, J4, J5, J6, L2, L3, Q2, R10, R11, R12, R13, R25, R26, R31, R32, R7, R9, RV1, SW1, U1, U10, U11, U14, U15, U2, U3, U7, U8, U9: LCSC (none) -> -
- D10, D3, D7, D8, D9: LCSC (none) -> C7420362
- R1, R2: LCSC (none) -> C7610430
- R14, R15, R16, R17, R19, R23: LCSC (none) -> C7319379
- R18, R20, R24, R27, R33, R34, R35, R36, R37: LCSC (none) -> C6654733
- R21, R22, R40, R41: LCSC (none) -> C7468408
- U4: LCSC C637131 -> -
- U5: LCSC (none) -> C7419972

Commit message: Update schematic
Parts:
- added C34: 100nF, Capacitor_SMD:C_0805_2012Metric, symbol Device:C
- L2: value 47uF -> 47uH; footprint Inductor_SMD:L_Bourns_SRP1038C_10.0x10.0mm -> Capacitor_SMD:C_2220_5750Metric
- Q2: footprint Package_TO_SOT_SMD:TO-263-2 -> Package_TO_SOT_SMD:TO-252-2
Connections:
- net +3.3V: now also C34.1
- net GND: now also C15.2, C9.2, R11.2, C34.2
