File: VFD-disp.kicad_pcb (KiCad board)
At the start: 4 copper layers, 99.6 x 65.5 mm, 118 parts, among them J1 USB_C_Receptacle_USB2.0_14P, J2 Conn_02x03_Odd_Even, J4 Conn_02x03_Odd_Even, J5 Conn_02x03_Odd_Even, J6 Conn_02x03_Odd_Even, Q1 Q_NMOS_GDS, Q2 Q_NMOS_GDS, Q3 Q_NPN_BEC, SW1 SW_SPST, U1 ESP32-C6-WROOM-1, U10 TXS0104EPW, U11 MAX811TEUS-T, U12 MCP4728, U13 TPS2116DRL, U14 KF50BDT, U15 AT24CS01-STUM, U2 FUSB302B01MPX, U3 LM1117DT-3.3, U4 MCP1416, U5 LM2576HVS-ADJ, U6 MAX1771xSA, U7 LM2576HVS-ADJ, U8 USBLC6-2P6, Y1 Crystal

Commit message: some changes
Parts:
- C1, C11, C12, C14, C17, C18, C19, C2, C20, C23, C26, C29, C3, C30, C33, C35, C36, C37, C4, C40, C41, C5, C8, C9: value C -> 100nF
- C10: value C -> Giga cap
- C13, C21, C22, C24, C25, C6: value C_Polarized -> 150uF
- C28, C34: value C_Polarized -> 40uF
- C31, C32: value C -> 200-600pF
- C7: value C_Polarized -> 10uF
- D1: value D -> B3100BE-13
- D2: value D_Zener -> Zener 3.5V
- D3, D4: value D_Schottky -> SS24
- F1: value Fuse -> 2A
- F4: value Fuse -> 500mA
- F5: value Fuse -> 750mA
- L1, L3, L4: value L -> 100uH
- R10: value R -> 10
- R11, R12, R14, R16, R29, R6: value R -> 10k
- R15, R17, R19, R30: value R -> 100k
- R18, R20, R24: value R -> 1k
- R21, R22, R3, R40, R41: value R -> 4.7k
- R4: value R -> 40m
- R5: value R -> 130k
- RV1, RV3: value R_Potentiometer -> 20k
- U7: value LM2576HVS-ADJ -> LM2576-5.0WU

Commit message: first working code
Parts:
- R23: value R -> 3.83k
- R27: value R -> 1k
- R28: value R -> 4.7k
- R9: value R -> 0R
Changed lines of the file:
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@@
 			)
 		)
-		(property "Value" "R"
+		(property "Value" "0R"
 			(at 0 1.65 0)
 			(layer "F.Fab")
@@
 			)
 		)
-		(property "Value" "R"
+		(property "Value" "1k"
 			(at 0 1.65 90)
 			(layer "F.Fab")
@@
 			)
 		)
-		(property "Value" "R"
+		(property "Value" "4.7k"
 			(at 0 1.65 0)
 			(layer "F.Fab")
@@
 			)
 		)
-		(property "Value" "R"
+		(property "Value" "3.83k"
 			(at 0 1.65 90)
 			(layer "F.Fab")

Commit message: update PCB with fixed values
Parts:
- R1, R2: value R -> 0R
- R5: value 130k -> 2.7k
- R6: value 10k -> 1.2k
- R9: value 0R -> R
Connections:
- U10 pad 8: GND -> +3.3V
Routing:
- net +3.3V: track 50.7 -> 58.1 mm
- net GND: track 188.1 -> 187.6 mm, vias 119 -> 118
Changed lines of the file:
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@@
 			)
 		)
-		(property "Value" "R"
+		(property "Value" "0R"
 			(at 0 1.65 90)
 			(layer "F.Fab")
@@
 			)
 		)
-		(property "Value" "0R"
+		(property "Value" "R"
 			(at 0 1.65 0)
 			(layer "F.Fab")
@@
 			)
 		)
-		(attr smd exclude_from_bom)
+		(attr smd exclude_from_bom dnp)
 		(duplicate_pad_numbers_are_jumpers no)
 		(fp_line
@@
 			)
 		)
-		(property "Value" "130k"
+		(property "Value" "2.7k"
 			(at 0 1.65 0)
 			(layer "F.Fab")
@@
 			(layers "F.Cu" "F.Mask" "F.Paste")
 			(roundrect_rratio 0.25)
-			(net "GND")
+			(net "+3.3V")
 			(pinfunction "OE_8")
 			(pintype "input")
@@
 			)
 		)
-		(property "Value" "10k"
+		(property "Value" "1.2k"
 			(at 0 1.65 0)
 			(layer "F.Fab")
@@
 			)
 		)
-		(property "Value" "R"
+		(property "Value" "0R"
 			(at 0 1.65 0)
 			(layer "F.Fab")
@@
 	)
 	(segment
-		(start 86.6 232)
-		(end 86.15 232)
-		(width 0.2)
-		(layer "F.Cu")
-		(net "GND")
-	)
-	(segment
 		(start 99.85 198.77)
 		(end 100.08 198.54)
@@
 	)
 	(segment
-		(start 86.15 232)
-		(end 86.14 232.01)
-		(width 0.2)
-		(layer "F.Cu")
-		(net "GND")
-	)
-	(segment
 		(start 98.75 210.15)
 		(end 98.725 210.15)
@@
 	)
 	(via
-		(at 86.14 232.01)
-		(size 0.45)
-		(drill 0.2)
-		(layers "F.Cu" "B.Cu")
-		(capping no)
-		(covering
-			(front no)
-			(back no)
-		)
-		(plugging
-			(front no)
-			(back no)
-		)
-		(filling no)
-		(net "GND")
-	)
-	(via
 		(at 106.35 197.94)
 		(size 0.8)
@@
 	)
 	(segment
+		(start 90.5 226.860246)
+		(end 90.5 226.275)
+		(width 0.2)
+		(layer "F.Cu")
+		(net "+3.3V")
+	)
+	(segment
 		(start 88.6 204.8)
 		(end 87.93 204.8)
@@
 	)
 	(segment
+		(start 86.6 230.760246)
+		(end 90.5 226.860246)
+		(width 0.2)
+		(layer "F.Cu")
+		(net "+3.3V")
+	)
+	(segment
 		(start 121.83 211.51)
 		(end 121.85 211.53)
@@
 		(width 0.2)
 		(layer "F.Cu")
+		(net "+3.3V")
+	)
+	(segment
+		(start 86.6 232)
+		(end 86.6 230.760246)
+		(width 0.2)
+		(layer "F.Cu")

Commit message: Rev 2 of schematic
Parts:
- removed C34: 40uF, Capacitor_Tantalum_SMD:CP_EIA-7343-31_Kemet-D
- removed Q2: Q_NMOS_GDS, Package_TO_SOT_SMD:TO-263-2
- removed R10: 10, Resistor_SMD:R_0805_2012Metric
- removed R11, R12: 10k, Resistor_SMD:R_0805_2012Metric
- removed U4: MCP1416, Package_TO_SOT_SMD:SOT-23-5
- added D10: BZT52C3V3-7-F, Diode_SMD:D_SOD-123, F.Cu at (117.4, 245.4)
- added D5: BZT52C3V3-7-F, Diode_SMD:D_SOD-123, F.Cu at (117.4, 235.8)
- added D7: BZT52C3V3-7-F, Diode_SMD:D_SOD-123, F.Cu at (117.4, 238.2)
- added D8: BZT52C3V3-7-F, Diode_SMD:D_SOD-123, F.Cu at (117.4, 240.6)
- added D9: BZT52C3V3-7-F, Diode_SMD:D_SOD-123, F.Cu at (117.4, 243.0)
- added R33: 1k, Resistor_SMD:R_0805_2012Metric, F.Cu at (113.0, 235.8)
- added R34: 1k, Resistor_SMD:R_0805_2012Metric, F.Cu at (113.0, 238.2)
- added R35: 1k, Resistor_SMD:R_0805_2012Metric, F.Cu at (113.0, 243.0)
- added R36: 1k, Resistor_SMD:R_0805_2012Metric, F.Cu at (113.0, 240.6)
- added R37: 1k, Resistor_SMD:R_0805_2012Metric, F.Cu at (113.0, 245.4)
- added U9: DRV8837, Package_SON:WSON-8-1EP_2x2mm_P0.5mm_EP0.9x1.6mm, F.Cu at (57.9, 246.8)
- moved C2 11.7 mm to (86.8, 238.6)
- moved C1 11.7 mm to (86.9, 246.8)
- moved HV5812WG1 11.7 mm to (76.4, 242.2)
- moved HV5812WG2 11.7 mm to (97.4, 242.2)
- moved C3 11.2 mm to (108.3, 245.1)
- moved C4 11.1 mm to (108.5, 237.1)
- moved C33 10.2 mm to (55.5, 246.8)
Connections:
- C33 pad 1: +5V -> +3.3V
- HV5812WG2 pad 10: G2 -> Net-(HV5812WG2-OUT13)
- HV5812WG2 pad 11: G1 -> Net-(HV5812WG2-OUT12)
- HV5812WG2 pad 7: G5 -> Net-(HV5812WG2-OUT16)
- HV5812WG2 pad 8: G4 -> Net-(HV5812WG2-OUT15)
- HV5812WG2 pad 9: G3 -> Net-(HV5812WG2-OUT14)
- R1 pad 2: F -> Net-(U9-OUT1)
- R2 pad 2: F -> Net-(U9-OUT1)
Routing:
- net Net-(D2-K): track 124.3 -> 19.0 mm
- net GREEN1: track 103.3 -> 0.00 mm, vias 1 -> 0
- net GREEN2: track 94.8 -> 0.00 mm, vias 1 -> 0
- net GREEN3: track 77.3 -> 0.00 mm, vias 1 -> 0
- net GREEN4: track 74.2 -> 0.00 mm, vias 1 -> 0
- net F_PWM: track 67.4 -> 0.00 mm, vias 2 -> 0
- net GREEN7: track 56.4 -> 0.00 mm, vias 1 -> 0
- net GREEN5: track 53.5 -> 0.00 mm, vias 1 -> 0
- net GREEN6: track 50.7 -> 0.00 mm, vias 1 -> 0
- net RED7: track 35.7 -> 0.00 mm, vias 1 -> 0
- net CLOCK: track 46.9 -> 14.9 mm
- net BLUE7: track 29.6 -> 0.00 mm, vias 1 -> 0
- net STROBE: track 52.7 -> 24.1 mm
- net RED6: track 24.2 -> 0.00 mm, vias 1 -> 0
- net BLANKING: track 29.7 -> 6.38 mm, vias 2 -> 0
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
Commit message: run autoroute
Routing:
- net Net-(U9-OUT1): track 0.00 -> 124.8 mm, vias 0 -> 2
- net GREEN1: track 0.00 -> 87.7 mm, vias 0 -> 1
- net GREEN2: track 0.00 -> 81.9 mm, vias 0 -> 1
- net F: track 61.9 -> 138.8 mm
- net GREEN3: track 0.00 -> 65.4 mm, vias 0 -> 1
- net F_PWM: track 0.00 -> 65.3 mm, vias 0 -> 4
- net Net-(D2-K): track 19.0 -> 83.6 mm, vias 0 -> 2
- net GND: track 174.4 -> 228.8 mm, vias 107 -> 109
- net +3.3V: track 54.5 -> 108.0 mm, vias 20 -> 22
- net GREEN4: track 0.00 -> 51.4 mm, vias 0 -> 1
- net GREEN7: track 0.00 -> 44.2 mm, vias 0 -> 1
- net F_EN: track 53.9 -> 97.6 mm, vias 2 -> 4
- net GREEN6: track 0.00 -> 39.9 mm, vias 0 -> 1
- net GREEN5: track 0.00 -> 38.3 mm, vias 0 -> 1
- net RED5: track 0.00 -> 29.8 mm, vias 0 -> 1
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